Commit message: daily update

File: dofbot.URDF (robot description, URDF)
Before this commit: robot dofbot, 7 links, 6 joints
Links:
- link base_link: geometry collision mesh filename=/home/ihpc-zrq/kan_ik/meshes/base_link.STL; visual mesh filename=/home/ihpc-zrq/kan_ik/meshes/base_link.STL
- link link1: geometry collision mesh filename=/home/ihpc-zrq/kan_ik/meshes/link1.STL; visual mesh filename=/home/ihpc-zrq/kan_ik/meshes/link1.STL
- link link2: geometry collision mesh filename=/home/ihpc-zrq/kan_ik/meshes/link2.STL; visual mesh filename=/home/ihpc-zrq/kan_ik/meshes/link2.STL
- link link3: geometry collision mesh filename=/home/ihpc-zrq/kan_ik/meshes/link3.STL; visual mesh filename=/home/ihpc-zrq/kan_ik/meshes/link3.STL
- link link4: geometry collision mesh filename=/home/ihpc-zrq/kan_ik/meshes/link4.STL; visual mesh filename=/home/ihpc-zrq/kan_ik/meshes/link4.STL
